Commit message: slider controller working

File: ur5_description/urdf/gazebo.xacro (robot description, xacro)
@@ -1,12 +1,11 @@
 <?xml version="1.0"?>
 <robot xmlns:xacro="http://www.ros.org/wiki/xacro" name="ur5_with_gripper">
-  <xacro:arg name="is_ignition" default="true"/>
-  <!-- ROS 2 Humble -->
+  <!-- IgnitionROS2Control plugin — loaded by gz_sim when the robot is spawned -->
   <gazebo>
-    <xacro:if value="$(arg is_ignition)">
-      <plugin filename="ign_ros2_control-system" name="ign_ros2_control::IgnitionROS2ControlPlugin">
-        <parameters>$(find ur5_controller)/config/controllers.yaml</parameters>
-      </plugin>
-    </xacro:if>
+    <plugin filename="ign_ros2_control-system"
+            name="ign_ros2_control::IgnitionROS2ControlPlugin">
+      <!-- Must match the YAML filename installed by ur5_controller -->
+      <parameters>$(find ur5_controller)/config/ur5_controllers.yaml</parameters>
+    </plugin>
   </gazebo>
 </robot>

File: ur5_description/urdf/inc/ur_joint_control.xacro (robot description, xacro)
@@ -1,4 +1,13 @@
 <?xml version="1.0"?>
 <robot xmlns:xacro="http://wiki.ros.org/xacro">
+  <!--
+    ros2_control joint interface definitions for the UR5 arm.
+    Only position command + position/velocity state interfaces are declared.
+    Velocity and effort command interfaces are removed: declaring interfaces
+    that no loaded controller claims causes IgnitionSystem to emit warnings on
+    every update cycle and can delay joint-state initialisation.
+    If you later add a velocity or effort controller, re-add the corresponding
+    <command_interface> here.
+  -->
   <xacro:macro name="ur_joint_control_description" params="
     tf_prefix
@@ -7,8 +16,5 @@
     <joint name="${tf_prefix}shoulder_pan_joint">
       <command_interface name="position"/>
-      <command_interface name="velocity"/>
-      <command_interface name="effort"/>
       <state_interface name="position">
-        <!-- initial position for the mock system and simulation -->
         <param name="initial_value">${initial_positions['shoulder_pan_joint']}</param>
       </state_interface>
@@ -16,14 +22,8 @@
         <param name="initial_value">0.0</param>
       </state_interface>
-      <state_interface name="effort">
-        <param name="initial_value">0.0</param>
-      </state_interface>
     </joint>
     <joint name="${tf_prefix}shoulder_lift_joint">
       <command_interface name="position"/>
-      <command_interface name="velocity"/>
-      <command_interface name="effort"/>
       <state_interface name="position">
-        <!-- initial position for the mock system and simulation -->
         <param name="initial_value">${initial_positions['shoulder_lift_joint']}</param>
       </state_interface>
@@ -31,14 +31,8 @@
         <param name="initial_value">0.0</param>
       </state_interface>
-      <state_interface name="effort">
-        <param name="initial_value">0.0</param>
-      </state_interface>
     </joint>
     <joint name="${tf_prefix}elbow_joint">
       <command_interface name="position"/>
-      <command_interface name="velocity"/>
-      <command_interface name="effort"/>
       <state_interface name="position">
-        <!-- initial position for the mock system and simulation -->
         <param name="initial_value">${initial_positions['elbow_joint']}</param>
       </state_interface>
@@ -46,14 +40,8 @@
         <param name="initial_value">0.0</param>
       </state_interface>
-      <state_interface name="effort">
-        <param name="initial_value">0.0</param>
-      </state_interface>
     </joint>
     <joint name="${tf_prefix}wrist_1_joint">
       <command_interface name="position"/>
-      <command_interface name="velocity"/>
-      <command_interface name="effort"/>
       <state_interface name="position">
-        <!-- initial position for the mock system and simulation -->
         <param name="initial_value">${initial_positions['wrist_1_joint']}</param>
       </state_interface>
@@ -61,14 +49,8 @@
         <param name="initial_value">0.0</param>
       </state_interface>
-      <state_interface name="effort">
-        <param name="initial_value">0.0</param>
-      </state_interface>
     </joint>
     <joint name="${tf_prefix}wrist_2_joint">
       <command_interface name="position"/>
-      <command_interface name="velocity"/>
-      <command_interface name="effort"/>
       <state_interface name="position">
-        <!-- initial position for the mock system and simulation -->
         <param name="initial_value">${initial_positions['wrist_2_joint']}</param>
       </state_interface>
@@ -76,14 +58,8 @@
         <param name="initial_value">0.0</param>
       </state_interface>
-      <state_interface name="effort">
-        <param name="initial_value">0.0</param>
-      </state_interface>
     </joint>
     <joint name="${tf_prefix}wrist_3_joint">
       <command_interface name="position"/>
-      <command_interface name="velocity"/>
-      <command_interface name="effort"/>
       <state_interface name="position">
-        <!-- initial position for the mock system and simulation -->
         <param name="initial_value">${initial_positions['wrist_3_joint']}</param>
       </state_interface>
@@ -91,7 +67,4 @@
         <param name="initial_value">0.0</param>
       </state_interface>
-      <state_interface name="effort">
-        <param name="initial_value">0.0</param>
-      </state_interface>
     </joint>
   </xacro:macro>

File: ur5_description/urdf/ros2_control_mock_hardware.xacro (robot description, xacro)
@@ -2,26 +2,49 @@
 <robot xmlns:xacro="http://www.ros.org/wiki/xacro">
   <xacro:include filename="$(find ur5_description)/urdf/inc/ur_joint_control.xacro" />
-  <xacro:include filename="$(find ur5_description)/urdf/inc/ur_sensors.xacro" />
+  <!--
+    ros2_control block for Ignition Gazebo (ign_ros2_control / ROS 2 Humble).
+    Plugin: ign_ros2_control/IgnitionSystem
+      - Reads joint states from the Ignition physics engine
+      - Writes position commands back into Ignition
+      - This is what makes the arm hold its position and respond to
+        JointTrajectory commands from arm_controller.
+    DO NOT add the fake FTS / TCP-pose sensors from ur_sensors.xacro here.
+    IgnitionSystem does not implement those state interfaces; including them
+    causes "[WARN] state interface not found" on every tick and can prevent
+    the system from initialising joint states correctly.
+  -->
   <xacro:macro name="ur_ros2_control" params="
     name
     tf_prefix
-    mock_sensor_commands:=false
     initial_positions:=${dict(shoulder_pan_joint=0.0,shoulder_lift_joint=-1.57,elbow_joint=0.0,wrist_1_joint=-1.57,wrist_2_joint=0.0,wrist_3_joint=0.0)}
     ">
     <ros2_control name="${name}" type="system">
       <hardware>
-        <!-- <plugin>mock_components/GenericSystem</plugin> -->
         <plugin>ign_ros2_control/IgnitionSystem</plugin>
-        <!-- <param name="mock_sensor_commands">${mock_sensor_commands}</param> -->
-        <!-- <param name="state_following_offset">0.0</param> -->
-        <!-- <param name="calculate_dynamics">true</param> -->
       </hardware>
+      <!-- UR5 arm — 6 DOF revolute joints -->
       <xacro:ur_joint_control_description
         tf_prefix="${tf_prefix}"
         initial_positions="${initial_positions}"
       />
-      <xacro:ur_sensors
-        tf_prefix="${tf_prefix}"
-      />
+      <!--
+        Robotiq 2F-85 — only the actuated finger_joint goes into ros2_control.
+        The 5 mimic joints (left/right inner/outer knuckle+finger) are purely
+        kinematic; robot_state_publisher propagates them from finger_joint via
+        the <mimic> tags in the URDF.  Putting them here would cause
+        "duplicate joint" errors.
+      -->
+      <joint name="${tf_prefix}finger_joint">
+        <command_interface name="position">
+          <param name="min">0.0</param>
+          <param name="max">0.725</param>
+        </command_interface>
+        <state_interface name="position">
+          <param name="initial_value">0.0</param>
+        </state_interface>
+        <state_interface name="velocity">
+          <param name="initial_value">0.0</param>
+        </state_interface>
+      </joint>
     </ros2_control>
   </xacro:macro>

File: ur5_description/urdf/ur5_with_gripper.urdf.xacro (robot description, xacro)
@@ -1,43 +1,62 @@
 <?xml version="1.0"?>
 <robot xmlns:xacro="http://wiki.ros.org/xacro" name="ur5_with_gripper">
-   <!-- Robot name parameter -->
-   <xacro:arg name="name" default="ur5"/>
-   <xacro:arg name="ur_type" default="ur5"/>
-   <xacro:arg name="tf_prefix" default=""/>
-   <!-- Import main UR macro -->
-   <xacro:include filename="$(find ur5_description)/urdf/ur_macro.xacro"/>
-   <!-- Import gripper macro -->
-   <!-- <xacro:include filename="$(find ur5_description)/urdf/robotiq_2f85_gripper.xacro"/> -->
-    <xacro:include filename="$(find ur5_description)/urdf/robotiq_arg85_gripper_macro.xacro"/>
-   <!-- Parameters -->
-   <xacro:arg name="joint_limit_params" default="$(find ur5_description)/config/$(arg ur_type)/joint_limits.yaml"/>
-   <xacro:arg name="kinematics_params" default="$(find ur5_description)/config/$(arg ur_type)/default_kinematics.yaml"/>
-   <xacro:arg name="physical_params" default="$(find ur5_description)/config/$(arg ur_type)/physical_parameters.yaml"/>
-   <xacro:arg name="visual_params" default="$(find ur5_description)/config/$(arg ur_type)/visual_parameters.yaml"/>
-   <xacro:arg name="transmission_hw_interface" default=""/>
-   <xacro:arg name="safety_limits" default="false"/>
-   <xacro:arg name="safety_pos_margin" default="0.15"/>
-   <xacro:arg name="safety_k_position" default="20"/>
-   <xacro:arg name="force_abs_paths" default="false"/>
-   <!-- Create world link -->
-   <link name="world"/>
-   <!-- UR5 Arm -->
-   <xacro:ur_robot
-     name="$(arg name)"
-     tf_prefix="$(arg tf_prefix)"
-     parent="world"
-     joint_limits_parameters_file="$(arg joint_limit_params)"
-     kinematics_parameters_file="$(arg kinematics_params)"
-     physical_parameters_file="$(arg physical_params)"
-     visual_parameters_file="$(arg visual_params)"
-     safety_limits="$(arg safety_limits)"
-     safety_pos_margin="$(arg safety_pos_margin)"
-     safety_k_position="$(arg safety_k_position)"
-     force_abs_paths="$(arg force_abs_paths)">
-     <origin xyz="0 0 0" rpy="0 0 0"/>
-   </xacro:ur_robot>
-   <!-- Add Robotiq 2F-85 Gripper -->
-   <xacro:robotiq_2f85_gripper prefix="" parent="tool0">
-     <origin xyz="0 0 0" rpy="0 0 0"/>
-   </xacro:robotiq_2f85_gripper>
+  <!-- ────────────────────────────────────────────────────────────────
+       Arguments
+  ──────────────────────────────────────────────────────────────────── -->
+  <xacro:arg name="name"                    default="ur5"/>
+  <xacro:arg name="ur_type"                 default="ur5"/>
+  <xacro:arg name="tf_prefix"               default=""/>
+  <xacro:arg name="joint_limit_params"      default="$(find ur5_description)/config/$(arg ur_type)/joint_limits.yaml"/>
+  <xacro:arg name="kinematics_params"       default="$(find ur5_description)/config/$(arg ur_type)/default_kinematics.yaml"/>
+  <xacro:arg name="physical_params"         default="$(find ur5_description)/config/$(arg ur_type)/physical_parameters.yaml"/>
+  <xacro:arg name="visual_params"           default="$(find ur5_description)/config/$(arg ur_type)/visual_parameters.yaml"/>
+  <xacro:arg name="safety_limits"           default="false"/>
+  <xacro:arg name="safety_pos_margin"       default="0.15"/>
+  <xacro:arg name="safety_k_position"       default="20"/>
+  <xacro:arg name="force_abs_paths"         default="false"/>
+  <!-- ────────────────────────────────────────────────────────────────
+       Includes
+  ──────────────────────────────────────────────────────────────────── -->
+  <!-- Kinematic / visual model -->
+  <xacro:include filename="$(find ur5_description)/urdf/ur_macro.xacro"/>
+  <!-- Robotiq 2F-85 gripper -->
+  <xacro:include filename="$(find ur5_description)/urdf/robotiq_arg85_gripper_macro.xacro"/>
+  <!-- ros2_control block (IgnitionSystem + joint definitions) -->
+  <xacro:include filename="$(find ur5_description)/urdf/ros2_control_mock_hardware.xacro"/>
+  <!-- Gazebo plugin (IgnitionROS2ControlPlugin) -->
+  <xacro:include filename="$(find ur5_description)/urdf/gazebo.xacro"/>
+  <!-- ────────────────────────────────────────────────────────────────
+       World link
+  ──────────────────────────────────────────────────────────────────── -->
+  <link name="world"/>
+  <!-- ────────────────────────────────────────────────────────────────
+       UR5 arm
+  ──────────────────────────────────────────────────────────────────── -->
+  <xacro:ur_robot
+    name="$(arg name)"
+    tf_prefix="$(arg tf_prefix)"
+    parent="world"
+    joint_limits_parameters_file="$(arg joint_limit_params)"
+    kinematics_parameters_file="$(arg kinematics_params)"
+    physical_parameters_file="$(arg physical_params)"
+    visual_parameters_file="$(arg visual_params)"
+    safety_limits="$(arg safety_limits)"
+    safety_pos_margin="$(arg safety_pos_margin)"
+    safety_k_position="$(arg safety_k_position)"
+    force_abs_paths="$(arg force_abs_paths)">
+    <origin xyz="0 0 0" rpy="0 0 0"/>
+  </xacro:ur_robot>
+  <!-- ────────────────────────────────────────────────────────────────
+       Robotiq 2F-85 gripper  (attached to tool0)
+  ──────────────────────────────────────────────────────────────────── -->
+  <xacro:robotiq_2f85_gripper prefix="" parent="tool0">
+    <origin xyz="0 0 0" rpy="0 0 0"/>
+  </xacro:robotiq_2f85_gripper>
+  <!-- ────────────────────────────────────────────────────────────────
+       ros2_control  (joints + IgnitionSystem hardware plugin)
+  ──────────────────────────────────────────────────────────────────── -->
+  <xacro:ur_ros2_control
+    name="$(arg name)"
+    tf_prefix="$(arg tf_prefix)"
+  />
 </robot>

File: ur5_description/urdf/ur_macro.xacro (robot description, xacro)
@@ -3,42 +3,7 @@
   <!--
     Base UR robot series xacro macro.
-    NOTE this is NOT a URDF. It cannot directly be loaded by consumers
-    expecting a flattened '.urdf' file. See the top-level '.xacro' for that
-    (but note that .xacro must still be processed by the xacro command).
-    This file models the base kinematic chain of a UR robot, which then gets
-    parameterised by various configuration files to convert it into a UR3(e),
-    UR5(e), UR10(e) or UR16e, etc.
-    NOTE the default kinematic parameters (i.e., link lengths, frame locations,
-    offsets, etc) do not correspond to any particular robot. They are defaults
-    only. There WILL be non-zero offsets between the Forward Kinematics results
-    in TF (i.e., robot_state_publisher) and the values reported by the Teach
-    Pendant.
-    For accurate (and robot-specific) transforms, the 'kinematics_parameters_file'
-    parameter MUST point to a .yaml file containing the appropriate values for
-    the targeted robot.
-    If using the UniversalRobots/Universal_Robots_ROS_Driver, follow the steps
-    described in the readme of that repository to extract the kinematic
-    calibration from the controller and generate the required .yaml file.
-    Main author of the migration to yaml configs Ludovic Delval.
-    Contributors to previous versions (in no particular order)
-     - Denis Stogl
-     - Lovro Ivanov
-     - Felix Messmer
-     - Kelsey Hawkins
-     - Wim Meeussen
-     - Shaun Edwards
-     - Nadia Hammoudeh Garcia
-     - Dave Hershberger
-     - G. vd. Hoorn
-     - Philip Long
-     - Dave Coleman
-     - Miguel Prada
-     - Mathias Luedtke
-     - Marcel Schnirring
-     - Felix von Drigalski
-     - Felix Exner
-     - Jimmy Da Silva
-     - Ajit Krisshna N L
-     - Muhammad Asif Rana
+    Modified: added meaningful joint dynamics (damping/friction) so Ignition
+    physics holds the arm erect before/between trajectory commands.
+    Without nonzero damping the arm collapses under gravity immediately.
   -->
   <xacro:include filename="$(find ur5_description)/urdf/inc/ur_common.xacro" />
@@ -65,10 +30,4 @@
       force_abs_paths="${force_abs_paths}"/>
     <!-- links -  main serial chain -->
-    <!-- base_link serves as the root of the robot's kinematic tree. It follows REP-103
-        conventions (i.e., X+ forward, Y+ left, Z+ up).
-        Since some kinematic solvers forbid having inertia values attached to a root link, we've
-        added the base_link_inertia link that carries the visual, collision and inertia
-        information.
-    -->
     <link name="${tf_prefix}base_link"/>
     <link name="${tf_prefix}base_link_inertia">
@@ -123,5 +82,6 @@
             izz="${shoulder_inertia_izz}"
         />
-      </inertial>    </link>
+      </inertial>
+    </link>
     <link name="${tf_prefix}upper_arm_link">
       <xacro:get_visual_params name="upper_arm" type="mesh_offset"/>
@@ -289,11 +249,13 @@
       <parent link="${tf_prefix}base_link" />
       <child link="${tf_prefix}base_link_inertia" />
-      <!-- 'base_link' is REP-103 aligned (so X+ forward), while the internal
-           frames of the robot/controller have X+ pointing backwards.
-           Use the joint between 'base_link' and 'base_link_inertia' (a dummy
-           link/frame) to introduce the necessary rotation over Z (of pi rad).
-      -->
       <origin xyz="0 0 0" rpy="0 0 ${pi}" />
     </joint>
+    <!--
+      IMPORTANT: nonzero damping is essential in Ignition/Gazebo.
+      With damping=0 the joints have no resistance and the arm falls under
+      gravity the moment it spawns.  Real UR5 joints have high gear-ratio
+      braking; 100 N·m·s/rad is a reasonable approximation that keeps the
+      arm erect while still allowing the trajectory controller to move it.
+    -->
     <joint name="${tf_prefix}shoulder_pan_joint" type="revolute">
       <parent link="${tf_prefix}base_link_inertia" />
@@ -306,5 +268,5 @@
          <safety_controller soft_lower_limit="${shoulder_pan_lower_limit + safety_pos_margin}" soft_upper_limit="${shoulder_pan_upper_limit - safety_pos_margin}" k_position="${safety_k_position}" k_velocity="0.0"/>
       </xacro:if>
-      <dynamics damping="0" friction="0"/>
+      <dynamics damping="100.0" friction="0.1"/>
     </joint>
     <joint name="${tf_prefix}shoulder_lift_joint" type="revolute">
@@ -318,5 +280,5 @@
          <safety_controller soft_lower_limit="${shoulder_lift_lower_limit + safety_pos_margin}" soft_upper_limit="${shoulder_lift_upper_limit - safety_pos_margin}" k_position="${safety_k_position}" k_velocity="0.0"/>
       </xacro:if>
-      <dynamics damping="0" friction="0"/>
+      <dynamics damping="100.0" friction="0.1"/>
     </joint>
     <joint name="${tf_prefix}elbow_joint" type="revolute">
@@ -330,5 +292,5 @@
          <safety_controller soft_lower_limit="${elbow_joint_lower_limit + safety_pos_margin}" soft_upper_limit="${elbow_joint_upper_limit - safety_pos_margin}" k_position="${safety_k_position}" k_velocity="0.0"/>
       </xacro:if>
-      <dynamics damping="0" friction="0"/>
+      <dynamics damping="100.0" friction="0.1"/>
     </joint>
     <joint name="${tf_prefix}wrist_1_joint" type="revolute">
@@ -342,5 +304,5 @@
          <safety_controller soft_lower_limit="${wrist_1_lower_limit + safety_pos_margin}" soft_upper_limit="${wrist_1_upper_limit - safety_pos_margin}" k_position="${safety_k_position}" k_velocity="0.0"/>
       </xacro:if>
-      <dynamics damping="0" friction="0"/>
+      <dynamics damping="10.0" friction="0.1"/>
     </joint>
     <joint name="${tf_prefix}wrist_2_joint" type="revolute">
@@ -354,5 +316,5 @@
          <safety_controller soft_lower_limit="${wrist_2_lower_limit + safety_pos_margin}" soft_upper_limit="${wrist_2_upper_limit - safety_pos_margin}" k_position="${safety_k_position}" k_velocity="0.0"/>
       </xacro:if>
-      <dynamics damping="0" friction="0"/>
+      <dynamics damping="10.0" friction="0.1"/>
     </joint>
     <joint name="${tf_prefix}wrist_3_joint" type="${wrist_3_joint_type}">
@@ -374,5 +336,5 @@
         </xacro:if>
       </xacro:unless>
-      <dynamics damping="0" friction="0"/>
+      <dynamics damping="10.0" friction="0.1"/>
     </joint>
     <link name="${tf_prefix}ft_frame"/>
@@ -382,17 +344,12 @@
       <origin xyz="0 0 0" rpy="${pi} 0 0"/>
     </joint>
-    <!-- ROS-Industrial 'base' frame - base_link to UR 'Base' Coordinates transform -->
+    <!-- ROS-Industrial 'base' frame -->
     <link name="${tf_prefix}base"/>
     <joint name="${tf_prefix}base_link-base_fixed_joint" type="fixed">
-      <!-- Note the rotation over Z of pi radians - as base_link is REP-103
-           aligned (i.e., has X+ forward, Y+ left and Z+ up), this is needed
-           to correctly align 'base' with the 'Base' coordinate system of
-           the UR controller.
-      -->
       <origin xyz="0 0 0" rpy="0 0 ${pi}"/>
       <parent link="${tf_prefix}base_link"/>
       <child link="${tf_prefix}base"/>
     </joint>
-    <!-- ROS-Industrial 'flange' frame - attachment point for EEF models -->
+    <!-- ROS-Industrial 'flange' frame -->
     <link name="${tf_prefix}flange" />
     <joint name="${tf_prefix}wrist_3-flange" type="fixed">
@@ -401,8 +358,7 @@
       <origin xyz="0 0 0" rpy="0 ${-pi/2.0} ${-pi/2.0}" />
     </joint>
-    <!-- ROS-Industrial 'tool0' frame - all-zeros tool frame -->
+    <!-- ROS-Industrial 'tool0' frame -->
     <link name="${tf_prefix}tool0"/>
     <joint name="${tf_prefix}flange-tool0" type="fixed">
-      <!-- default toolframe - X+ left, Y+ up, Z+ front -->
       <origin xyz="0 0 0" rpy="${pi/2.0} 0 ${pi/2.0}"/>
       <parent link="${tf_prefix}flange"/>
